Commit message: put gripper with dummy joint into xacros

File: euler_support/urdf/eef_macro.xacro (robot description, xacro)
@@ -23,4 +23,5 @@
     </link>
     <link name="${prefix}tcp"/>
+    <link name="${prefix}eef_link"/>
     <joint name="${prefix}eef_base_to_${prefix}eef_body" type="fixed">
       <parent link="${prefix}eef_base" />
@@ -33,4 +34,11 @@
       <origin xyz="0 0 0.17" rpy="0 0 0" />
     </joint>
+    <joint name="motoman_eef_joint" type="revolute">
+      <parent link="${prefix}eef_body" />
+      <child link="${prefix}eef_link" />
+      <origin xyz="0 0 0" rpy="0 0 0" />
+      <axis xyz="0 0 1" />
+      <limit lower="-1" upper="1" effort="10" velocity="100" />
+    </joint>
   </xacro:macro>
 </robot>

File: euler_support/urdf/euler_macro.xacro (robot description, xacro)
@@ -11,5 +11,5 @@
         <!--xacro:asus_xtion_pro sensor_name="" off_x="0.461" off_y="0" off_z="2.103" off_rr="1.5708" off_rp="1.8849" off_ry="0"/-->
         <xacro:asus_sensor_definitions prefix="asus" parent_link="motoman_base_link" />
-        <!--<xacro:eef prefix=""/>-->
+        <xacro:eef prefix=""/>
         <!--link list -->
         <link name="${prefix}base_link"> </link>
@@ -165,9 +165,9 @@
                 <axis xyz="0 0 0" />
         </joint>
-        <!--<joint name="motoman_link_t_to_eef_base" type="fixed">
+        <joint name="motoman_link_t_to_eef_base" type="fixed">
                 <parent link="motoman_link_t" />
                 <child link="eef_base" />
                 <origin xyz="0.098 0 0" rpy="0 1.57 0" />
-        </joint>-->
+        </joint>
 </xacro:macro>
 </robot>
